Commit message: 第二版urdf模型webots中可以轨迹跟随

File: src/assembly_robot/resource/asmb_robot.urdf (robot description, URDF)
Before this commit: robot asmb_robot, 20 links, 19 joints
Links:
- added link base_footprint
Joints:
- added joint base_joint: type fixed, parent base_footprint, child base_link, origin xyz=0.0 0.0 0.01 rpy=0 0 0
