Commit message: 修改部分文件路径

File: src/assembly_robot/urdf/asmb_robot.urdf (robot description, URDF)
Before this commit: robot asmb_robot, 15 links, 14 joints
Links:
- added link base_footprint
Joints:
- added joint base_joint: type fixed, parent base_footprint, child base_link, origin xyz=0.0 0.0 0.6 rpy=0 0 0

Commit message: 更换新的urdf文件后 nodes.py运行报错

File: src/assembly_robot/urdf/asmb_robot.urdf (robot description, URDF)
Before this commit: robot asmb_robot, 16 links, 15 joints
Links:
- removed link base_footprint
- removed link left_arm_link1
- removed link left_arm_link2
- removed link left_arm_link3
- removed link left_arm_link4
- removed link left_arm_link5
- removed link left_arm_link6
- removed link right_arm_link1
- removed link right_arm_link2
- removed link right_arm_link3
- removed link right_arm_link4
- removed link right_arm_link5
- removed link right_arm_link6
- removed link right_arm_link7
- added link head_camera_Link, mass 0.061182; collision mesh filename=package://assembly_robot/resource/asmb_robot/meshes/head_ca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; visual mesh filename=package://assembly_robot/resource/asmb_robot/meshes/head_ca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
- added link left_arm_Link1, mass 0; collision mesh filename=package://assembly_robot/resource/asmb_robot/meshes/left_ar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; visual mesh filename=package://assembly_robot/resource/asmb_robot/meshes/left_ar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
- added link left_arm_Link2, mass 0.470284076871094; collision mesh filename=package://assembly_robot/resource/asmb_robot/meshes/left_ar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; visual mesh filename=package://assembly_robot/resource/asmb_robot/meshes/left_ar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
- added link left_arm_Link3, mass 0.129990371419528; collision mesh filename=package://assembly_robot/resource/asmb_robot/meshes/left_ar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; visual mesh filename=package://assembly_robot/resource/asmb_robot/meshes/left_ar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
- added link left_arm_Link4, mass 0.477207553120282; collision mesh filename=package://assembly_robot/resource/asmb_robot/meshes/left_ar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; visual mesh filename=package://assembly_robot/resource/asmb_robot/meshes/left_ar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
- added link left_arm_Link5, mass 0.114969387635768; collision mesh filename=package://assembly_robot/resource/asmb_robot/meshes/left_ar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; visual mesh filename=package://assembly_robot/resource/asmb_robot/meshes/left_ar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
- added link left_arm_Link6, mass 0.0852865509434714; collision mesh filename=package://assembly_robot/resource/asmb_robot/meshes/left_ar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; visual mesh filename=package://assembly_robot/resource/asmb_robot/meshes/left_ar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
- added link left_finger_link1, mass 0.0040452362516926; collision mesh filename=package://assembly_robot/resource/asmb_robot/meshes/left_fi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; visual mesh filename=package://assembly_robot/resource/asmb_robot/meshes/left_fi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
- added link left_finger_link2, mass 0.0040452362516926; collision mesh filename=package://assembly_robot/resource/asmb_robot/meshes/left_fi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; visual mesh filename=package://assembly_robot/resource/asmb_robot/meshes/left_fi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
- added link right_arm_Link1, mass 0.37147; collision mesh filename=package://assembly_robot/resource/asmb_robot/meshes/right_a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; visual mesh filename=package://assembly_robot/resource/asmb_robot/meshes/right_a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
- added link right_arm_Link2, mass 0.47028; collision mesh filename=package://assembly_robot/resource/asmb_robot/meshes/right_a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; visual mesh filename=package://assembly_robot/resource/asmb_robot/meshes/right_a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
- added link right_arm_Link3, mass 0.12999; collision mesh filename=package://assembly_robot/resource/asmb_robot/meshes/right_a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; visual mesh filename=package://assembly_robot/resource/asmb_robot/meshes/right_a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
- added link right_arm_Link4, mass 0.47713; collision mesh filename=package://assembly_robot/resource/asmb_robot/meshes/right_a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; visual mesh filename=package://assembly_robot/resource/asmb_robot/meshes/right_a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
- added link right_arm_Link5, mass 0.36518735117001; collision mesh filename=package://assembly_robot/resource/asmb_robot/meshes/right_a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; visual mesh filename=package://assembly_robot/resource/asmb_robot/meshes/right_a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
- added link right_arm_Link6, mass 0.0772380702383185; collision mesh filename=package://assembly_robot/resource/asmb_robot/meshes/right_a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; visual mesh filename=package://assembly_robot/resource/asmb_robot/meshes/right_a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
- added link right_arm_Link7, mass 0.235933563807994; collision mesh filename=package://assembly_robot/resource/asmb_robot/meshes/right_a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; visual mesh filename=package://assembly_robot/resource/asmb_robot/meshes/right_a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
- added link right_finger_link1, mass 10.2661535963727; collision mesh filename=package://assembly_robot/resource/asmb_robot/meshes/right_f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; visual mesh filename=package://assembly_robot/resource/asmb_robot/meshes/right_f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
- added link right_finger_link2, mass 10.2661535963727; collision mesh filename=package://assembly_robot/resource/asmb_robot/meshes/right_f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; visual mesh filename=package://assembly_robot/resource/asmb_robot/meshes/right_f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
- link base_link: mass 6.0305 -> 5.9383
- link left_arm_link7: mass 0.246381268980238 -> 0.235933563807994
Joints:
- removed joint base_joint
- added joint head_camera_joint: type revolute, parent base_link, child head_camera_Link, origin xyz=0.0875 0.065 1.6145 rpy=0 0 0, axis 0 1 0, limit lower=-1.57 upper=1.57 effort=100 velocity=1
- added joint left_finger_joint1: type prismatic, parent left_arm_link7, child left_finger_link1, origin xyz=0 -0.013 -0.1435 rpy=0 0 0, axis 0 -1 0, limit lower=-0.013 upper=0 effort=100 velocity=1
- added joint left_finger_joint2: type prismatic, parent left_arm_link7, child left_finger_link2, origin xyz=0 0.013 -0.1435 rpy=0 0 0, axis 0 -1 0, limit lower=0 upper=0.013 effort=100 velocity=1
- added joint right_finger_joint1: type prismatic, parent right_arm_Link7, child right_finger_link1, origin xyz=0 0.013 -0.1435 rpy=0 0 0, axis 0 1 0, limit lower=-0.013 upper=0 effort=100 velocity=1
- added joint right_finger_joint2: type prismatic, parent right_arm_Link7, child right_finger_link2, origin xyz=0 -0.013 -0.1435 rpy=0 0 0, axis 0 1 0, limit lower=0 upper=0.013 effort=100 velocity=1
- joint left_arm_joint1: child left_arm_link1 -> left_arm_Link1; origin xyz=-0.1469 -0.1 0.473 rpy=0 0 1.5708 -> xyz=0 0.1469 1.319 rpy=0 0 0
- joint left_arm_joint2: axis 1 0 0 -> -1 0 0; child left_arm_link2 -> left_arm_Link2; limit lower=-3.14 upper=3.14 effort=100 velocity=1 -> lower=-3.14 upper=0 effort=100 velocity=1; origin xyz=-0.057 0.0536 0 rpy=0 0 0 -> xyz=0.057 0.0536 0 rpy=0 0 0; parent left_arm_link1 -> left_arm_Link1
- joint left_arm_joint3: child left_arm_link3 -> left_arm_Link3; origin xyz=0.057 0 -0.15815 rpy=0 0 0 -> xyz=-0.057 0 -0.15815 rpy=0 0 0; parent left_arm_link2 -> left_arm_Link2
- joint left_arm_joint4: child left_arm_link4 -> left_arm_Link4; limit lower=-3.14 upper=3.14 effort=100 velocity=1 -> lower=-1.57 upper=1.57 effort=100 velocity=1; parent left_arm_link3 -> left_arm_Link3
- joint left_arm_joint5: child left_arm_link5 -> left_arm_Link5; origin xyz=0 -0.052 -0.15815 rpy=0 0 0 -> xyz=0 -0.052 -0.162 rpy=0 0 0; parent left_arm_link4 -> left_arm_Link4
- joint left_arm_joint6: axis -1 0 0 -> 1 0 0; child left_arm_link6 -> left_arm_Link6; limit lower=-3.14 upper=3.14 effort=100 velocity=1 -> lower=-1.57 upper=1.57 effort=100 velocity=1; origin xyz=-0.04715 0 -0.07985 rpy=0 0 0 -> xyz=0.044 0 -0.076 rpy=0 0 0; parent left_arm_link5 -> left_arm_Link5
- joint left_arm_joint7: origin xyz=0.04715 0 -0.067 rpy=0 0 0 -> xyz=-0.044 0 -0.067 rpy=0 0 0; parent left_arm_link6 -> left_arm_Link6
- joint right_arm_joint1: child right_arm_link1 -> right_arm_Link1; origin xyz=0.1469 -0.1 0.473 rpy=0 0 1.5708 -> xyz=0 -0.1469 1.319 rpy=0 0 0
- joint right_arm_joint2: axis 1 0 0 -> -1 0 0; child right_arm_link2 -> right_arm_Link2; limit lower=-3.14 upper=3.14 effort=100 velocity=1 -> lower=0 upper=3.14 effort=100 velocity=1; origin xyz=-0.057 -0.0536 0 rpy=0 0 0 -> xyz=0.057 -0.0536 0 rpy=0 0 0; parent right_arm_link1 -> right_arm_Link1
- joint right_arm_joint3: child right_arm_link3 -> right_arm_Link3; origin xyz=0.057 0 -0.15815 rpy=0 0 0 -> xyz=-0.057 0 -0.15815 rpy=0 0 0; parent right_arm_link2 -> right_arm_Link2
- joint right_arm_joint4: child right_arm_link4 -> right_arm_Link4; limit lower=-3.14 upper=3.14 effort=100 velocity=1 -> lower=-1.57 upper=1.57 effort=100 velocity=1; parent right_arm_link3 -> right_arm_Link3
- joint right_arm_joint5: child right_arm_link5 -> right_arm_Link5; origin xyz=0 0.052 -0.162 rpy=0 0 0 -> xyz=0 0.052 -0.15815 rpy=0 0 0; parent right_arm_link4 -> right_arm_Link4
- joint right_arm_joint6: axis -1 0 0 -> 1 0 0; child right_arm_link6 -> right_arm_Link6; limit lower=-3.14 upper=3.14 effort=100 velocity=1 -> lower=-1.57 upper=1.57 effort=100 velocity=1; origin xyz=-0.044 0 -0.076 rpy=0 0 0 -> xyz=0.05 0 -0.07985 rpy=0 0 0; parent right_arm_link5 -> right_arm_Link5
- joint right_arm_joint7: child right_arm_link7 -> right_arm_Link7; origin xyz=0.044 0 -0.067 rpy=0 0 0 -> xyz=-0.05 0 -0.067 rpy=0 0 0; parent right_arm_link6 -> right_arm_Link6

Commit message: 第一版urdf模型webots中可以运动

File: src/assembly_robot/urdf/asmb_robot.urdf (robot description, URDF)
Before this commit: robot ASMBRobot, 20 links, 19 joints
Links:
- removed link head_camera_Link
- removed link left_arm_Link1
- removed link left_arm_Link2
- removed link left_arm_Link3
- removed link left_arm_Link4
- removed link left_arm_Link5
- removed link left_arm_Link6
- removed link left_finger_link1
- removed link left_finger_link2
- removed link right_arm_Link1
- removed link right_arm_Link2
- removed link right_arm_Link3
- removed link right_arm_Link4
- removed link right_arm_Link5
- removed link right_arm_Link6
- removed link right_arm_Link7
- removed link right_finger_link1
- removed link right_finger_link2
- added link base_footprint
- added link left_arm_link1, mass 0.37555886929927; collision mesh filename=package://assembly_robot/resource/asmb_robot/meshes/left_ar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; visual mesh filename=package://assembly_robot/resource/asmb_robot/meshes/left_ar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
- added link left_arm_link2, mass 0.471882858713434; collision mesh filename=package://assembly_robot/resource/asmb_robot/meshes/left_ar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; visual mesh filename=package://assembly_robot/resource/asmb_robot/meshes/left_ar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
- added link left_arm_link3, mass 0.134068404066203; collision mesh filename=package://assembly_robot/resource/asmb_robot/meshes/left_ar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; visual mesh filename=package://assembly_robot/resource/asmb_robot/meshes/left_ar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
- added link left_arm_link4, mass 0.481341653757711; collision mesh filename=package://assembly_robot/resource/asmb_robot/meshes/left_ar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; visual mesh filename=package://assembly_robot/resource/asmb_robot/meshes/left_ar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
- added link left_arm_link5, mass 0.36518735117001; collision mesh filename=package://assembly_robot/resource/asmb_robot/meshes/left_ar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; visual mesh filename=package://assembly_robot/resource/asmb_robot/meshes/left_ar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
- added link left_arm_link6, mass 0.0794420469377912; collision mesh filename=package://assembly_robot/resource/asmb_robot/meshes/left_ar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; visual mesh filename=package://assembly_robot/resource/asmb_robot/meshes/left_ar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
- added link right_arm_link1, mass 0.375354991700786; collision mesh filename=package://assembly_robot/resource/asmb_robot/meshes/right_a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; visual mesh filename=package://assembly_robot/resource/asmb_robot/meshes/right_a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
- added link right_arm_link2, mass 0.470914062127475; collision mesh filename=package://assembly_robot/resource/asmb_robot/meshes/right_a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; visual mesh filename=package://assembly_robot/resource/asmb_robot/meshes/right_a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
- added link right_arm_link3, mass 0.134068404066203; collision mesh filename=package://assembly_robot/resource/asmb_robot/meshes/right_a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; visual mesh filename=package://assembly_robot/resource/asmb_robot/meshes/right_a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
- added link right_arm_link4, mass 0.480553306375498; collision mesh filename=package://assembly_robot/resource/asmb_robot/meshes/right_a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; visual mesh filename=package://assembly_robot/resource/asmb_robot/meshes/right_a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
- added link right_arm_link5, mass 0.271897101050664; collision mesh filename=package://assembly_robot/resource/asmb_robot/meshes/right_a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; visual mesh filename=package://assembly_robot/resource/asmb_robot/meshes/right_a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
- added link right_arm_link6, mass 0.0864651823892207; collision mesh filename=package://assembly_robot/resource/asmb_robot/meshes/right_a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; visual mesh filename=package://assembly_robot/resource/asmb_robot/meshes/right_a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
- added link right_arm_link7, mass 0.226179539449807; collision mesh filename=package://assembly_robot/resource/asmb_robot/meshes/right_a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; visual mesh filename=package://assembly_robot/resource/asmb_robot/meshes/right_a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
- link base_link: mass 5.9383 -> 6.0305
- link left_arm_link7: mass 0.235933563807994 -> 0.246381268980238
Joints:
- removed joint head_camera_joint
- removed joint left_finger_joint1
- removed joint left_finger_joint2
- removed joint right_finger_joint1
- removed joint right_finger_joint2
- joint left_arm_joint1: child left_arm_Link1 -> left_arm_link1; origin xyz=0 0.1469 1.319 rpy=0 0 0 -> xyz=-0.1469 -0.1 0.473 rpy=0 0 1.5708
- joint left_arm_joint2: axis -1 0 0 -> 1 0 0; child left_arm_Link2 -> left_arm_link2; limit lower=-3.14 upper=0 effort=100 velocity=1 -> lower=-3.14 upper=3.14 effort=100 velocity=1; origin xyz=0.057 0.0536 0 rpy=0 0 0 -> xyz=-0.057 0.0536 0 rpy=0 0 0; parent left_arm_Link1 -> left_arm_link1
- joint left_arm_joint3: child left_arm_Link3 -> left_arm_link3; origin xyz=-0.057 0 -0.15815 rpy=0 0 0 -> xyz=0.057 0 -0.15815 rpy=0 0 0; parent left_arm_Link2 -> left_arm_link2
- joint left_arm_joint4: child left_arm_Link4 -> left_arm_link4; limit lower=-1.57 upper=1.57 effort=100 velocity=1 -> lower=-3.14 upper=3.14 effort=100 velocity=1; parent left_arm_Link3 -> left_arm_link3
- joint left_arm_joint5: child left_arm_Link5 -> left_arm_link5; origin xyz=0 -0.052 -0.162 rpy=0 0 0 -> xyz=0 -0.052 -0.15815 rpy=0 0 0; parent left_arm_Link4 -> left_arm_link4
- joint left_arm_joint6: axis 1 0 0 -> -1 0 0; child left_arm_Link6 -> left_arm_link6; limit lower=-1.57 upper=1.57 effort=100 velocity=1 -> lower=-3.14 upper=3.14 effort=100 velocity=1; origin xyz=0.044 0 -0.076 rpy=0 0 0 -> xyz=-0.04715 0 -0.07985 rpy=0 0 0; parent left_arm_Link5 -> left_arm_link5
- joint left_arm_joint7: origin xyz=-0.044 0 -0.067 rpy=0 0 0 -> xyz=0.04715 0 -0.067 rpy=0 0 0; parent left_arm_Link6 -> left_arm_link6
- joint right_arm_joint1: child right_arm_Link1 -> right_arm_link1; origin xyz=0 -0.1469 1.319 rpy=0 0 0 -> xyz=0.1469 -0.1 0.473 rpy=0 0 1.5708
- joint right_arm_joint2: axis -1 0 0 -> 1 0 0; child right_arm_Link2 -> right_arm_link2; limit lower=0 upper=3.14 effort=100 velocity=1 -> lower=-3.14 upper=3.14 effort=100 velocity=1; origin xyz=0.057 -0.0536 0 rpy=0 0 0 -> xyz=-0.057 -0.0536 0 rpy=0 0 0; parent right_arm_Link1 -> right_arm_link1
- joint right_arm_joint3: child right_arm_Link3 -> right_arm_link3; origin xyz=-0.057 0 -0.15815 rpy=0 0 0 -> xyz=0.057 0 -0.15815 rpy=0 0 0; parent right_arm_Link2 -> right_arm_link2
- joint right_arm_joint4: child right_arm_Link4 -> right_arm_link4; limit lower=-1.57 upper=1.57 effort=100 velocity=1 -> lower=-3.14 upper=3.14 effort=100 velocity=1; parent right_arm_Link3 -> right_arm_link3
- joint right_arm_joint5: child right_arm_Link5 -> right_arm_link5; origin xyz=0 0.052 -0.15815 rpy=0 0 0 -> xyz=0 0.052 -0.162 rpy=0 0 0; parent right_arm_Link4 -> right_arm_link4
- joint right_arm_joint6: axis 1 0 0 -> -1 0 0; child right_arm_Link6 -> right_arm_link6; limit lower=-1.57 upper=1.57 effort=100 velocity=1 -> lower=-3.14 upper=3.14 effort=100 velocity=1; origin xyz=0.05 0 -0.07985 rpy=0 0 0 -> xyz=-0.044 0 -0.076 rpy=0 0 0; parent right_arm_Link5 -> right_arm_link5
- joint right_arm_joint7: child right_arm_Link7 -> right_arm_link7; origin xyz=-0.05 0 -0.067 rpy=0 0 0 -> xyz=0.044 0 -0.067 rpy=0 0 0; parent right_arm_Link6 -> right_arm_link6
